Commit message: Human model now with right upper and lower arm.

File: urdf/human.urdf.xacro (robot description, xacro)
@@ -10,14 +10,22 @@
   <!-- Main Body-base -->
   <property name="depth" value="0.05" />
-  <property name="hips_length" value="0.107" />
+  <property name="hips_length" value="0.086" />
   <property name="hips_width" value="0.099" />
-  <property name="spine_length" value="0.257" />
+  <property name="spine_length" value="0.172" />
   <property name="shoulder_width" value="0.198" />
   <property name="neck_length" value="0.103" />
   <property name="head_size" value="0.05" />
+  <property name="upper_arm_length" value="0.159" />
+  <property name="arm_radius" value="0.025" />
+  <property name="trunk_length" value="0.258" />
+  <property name="lower_arm_length" value="0.143" />
   <link name="world"/>
   <link name="hips_dummy"/>
   <link name="head_dummy"/>
   <link name="head_dummy_2"/>
+  <link name="r_upper_arm_dummy"/>
+  <link name="r_upper_arm_dummy_2"/>
+  <link name="r_lower_arm_dummy"/>
+  <link name="r_lower_arm_dummy_2"/>
   <link name="hips">
     <visual>
@@ -42,16 +50,34 @@
       <origin xyz="0 0 0" rpy="0 0 0" />
       <geometry>
-        <cylinder length="${neck_length}" radius="${head_size}"/>"/>
+        <cylinder length="${neck_length}" radius="${head_size}"/>
       </geometry>
       <material name="White" />
     </visual>
   </link>
-  <joint name="hips_pitch" type="continuous">
-    <origin xyz="0 0 0" rpy="0 0 ${M_PI_2}" />
+  <link name="r_upper_arm">
+    <visual>
+      <origin xyz="0 0 ${-upper_arm_length/2}" rpy="0 0 0" />
+      <geometry>
+        <cylinder length="${upper_arm_length}" radius="${arm_radius}"/>
+      </geometry>
+      <material name="Black" />
+    </visual>
+  </link>
+  <link name="r_lower_arm">
+    <visual>
+      <origin xyz="0 0 ${-lower_arm_length/2}" rpy="0 0 0" />
+      <geometry>
+        <cylinder length="${lower_arm_length}" radius="${arm_radius}"/>
+      </geometry>
+      <material name="Gray" />
+    </visual>
+  </link>
+  <joint name="hips_p" type="continuous">
+    <origin xyz="0 0 0" rpy="0 0 0" />
     <parent link="world"/>
     <child link="hips" />
     <axis xyz="0 1 0" rpy="0 0 0" />
   </joint>
-  <joint name="hips_roll" type="continuous">
+  <joint name="hips_r" type="continuous">
     <origin xyz="0 0 0" rpy="0 0 0" />
     <parent link="hips"/>
@@ -59,5 +85,5 @@
     <axis xyz="1 0 0" rpy="0 0 0" />
   </joint>
-  <joint name="hips_yaw" type="continuous">
+  <joint name="hips_y" type="continuous">
     <origin xyz="0 0 ${hips_length/2 + spine_length/2}" rpy="0 0 0" />
     <parent link="hips_dummy"/>
@@ -65,5 +91,5 @@
     <axis xyz="0 0 1" rpy="0 0 0" />
   </joint>
-  <joint name="head_pitch" type="continuous">
+  <joint name="head_p" type="continuous">
     <origin xyz="0 0 ${spine_length/2+neck_length/2}" rpy="0 0 ${M_PI_2}" />
     <parent link="spine"/>
@@ -71,5 +97,5 @@
     <axis xyz="0 1 0" rpy="0 0 0" />
   </joint>
-  <joint name="head_roll" type="continuous">
+  <joint name="head_r" type="continuous">
     <origin xyz="0 0 0" rpy="0 0 0" />
     <parent link="head_dummy"/>
@@ -77,5 +103,5 @@
     <axis xyz="1 0 0" rpy="0 0 0" />
   </joint>
-  <joint name="head_yaw" type="continuous">
+  <joint name="head_y" type="continuous">
     <origin xyz="0 0 0" rpy="0 0 0" />
     <parent link="head_dummy_2"/>
@@ -83,3 +109,39 @@
     <axis xyz="0 0 1" rpy="0 0 0" />
   </joint>
+  <joint name="r_upper_arm_r" type="continuous">
+    <origin xyz="${-shoulder_width/2} 0 ${spine_length/2-arm_radius/2}" rpy="0 ${M_PI_2} 0" />
+    <parent link="spine"/>
+    <child link="r_upper_arm_dummy" />
+    <axis xyz="-1 0 0" rpy="0 0 0" />
+  </joint>
+  <joint name="r_upper_arm_p" type="continuous">
+    <origin xyz="0 0 0" rpy="0 0 0" />
+    <parent link="r_upper_arm_dummy"/>
+    <child link="r_upper_arm_dummy_2" />
+    <axis xyz="0 1 0" rpy="0 0 0" />
+  </joint>
+  <joint name="r_upper_arm_y" type="continuous">
+    <origin xyz="0 0 0" rpy="0 0 0" />
+    <parent link="r_upper_arm_dummy_2"/>
+    <child link="r_upper_arm" />
+    <axis xyz="0 0 -1" rpy="0 0 0" />
+  </joint>
+  <joint name="r_lower_arm_r" type="continuous">
+    <origin xyz="0 0 ${-upper_arm_length}" rpy="0 0 0" />
+    <parent link="r_upper_arm"/>
+    <child link="r_lower_arm_dummy" />
+    <axis xyz="-1 0 0" rpy="0 0 0" />
+  </joint>
+  <joint name="r_lower_arm_p" type="continuous">
+    <origin xyz="0 0 0" rpy="0 0 0" />
+    <parent link="r_lower_arm_dummy"/>
+    <child link="r_lower_arm_dummy_2" />
+    <axis xyz="0 1 0" rpy="0 0 0" />
+  </joint>
+  <joint name="r_lower_arm_y" type="continuous">
+    <origin xyz="0 0 0" rpy="0 0 0" />
+    <parent link="r_lower_arm_dummy_2"/>
+    <child link="r_lower_arm" />
+    <axis xyz="0 0 -1" rpy="0 0 0" />
+  </joint>
 </robot>
